Commit message: Add Marsdog style imitation task with multi-critic RL support.
Introduce the style task for cyclic gait imitation, extend reward and env managers for grouped critics, refresh Marsdog assets and motion data, and add motion tooling scripts.

Co-authored-by: Cursor <cursoragent@cursor.com>

File: src/mjlab/asset_zoo/robots/marsdog/xmls/assets/marsdog.urdf (robot description, URDF)
Before this commit: robot marsdog, 53 links, 52 joints
Links:
- removed link imu_link
- removed link tail10_link
- removed link tail10_virtual_link
- removed link tail11_link
- removed link tail11_virtual_link
- removed link tail12_link
- removed link tail12_virtual_link
- removed link tail1_link
- removed link tail1_virtual_link
- removed link tail2_link
- removed link tail2_virtual_link
- removed link tail3_link
- removed link tail3_virtual_link
- removed link tail4_link
- removed link tail4_virtual_link
- removed link tail5_link
- removed link tail5_virtual_link
- removed link tail6_link
- removed link tail6_virtual_link
- removed link tail7_link
- removed link tail7_virtual_link
- removed link tail8_link
- removed link tail8_virtual_link
- removed link tail9_link
- removed link tail9_virtual_link
- added link tail_pitch_link, mass 0.00601534; collision cylinder length=0.04 radius=0.009; visual mesh filename=package://marsdog/meshes/tail_pitch_link.STL
- added link tail_yaw_link, mass 0.00601534; collision cylinder length=0.02 radius=0.01; visual mesh filename=package://marsdog/meshes/tail_yaw_link.STL
- link base_link: mass 2.875 -> 1.43861788; geometry collision box size=0.14 0.065 0.08; collision cylinder length=0.05 radius=0.04
- link fl_calf_link: mass 0.462 -> 0.41615103; geometry collision cylinder length=0.05 radius=0.023; collision cylinder length=0.09 radius=0.016
- link fl_foot_link: mass 0.005 -> 0.00282686
- link fl_hip_pitch_link: mass 0.266 -> 0.19550425
- link fl_tarsus_link: mass 0.067 -> 0.09354472; geometry collision cylinder length=0.055 radius=0.018; visual mesh filename=package://marsdog/meshes/fl_tarsus_link.STL
- link fl_thigh_roll_link: mass 0.087 -> 0.08017506; geometry collision box size=0.01 0.035 0.07; visual mesh filename=package://marsdog/meshes/fl_thigh_roll_link.STL
- link fr_calf_link: mass 0.462 -> 0.41615103; geometry collision cylinder length=0.05 radius=0.023; collision cylinder length=0.09 radius=0.016
- link fr_foot_link: mass 0.005 -> 0.00282686
- link fr_hip_pitch_link: mass 0.266 -> 0.19550425
- link fr_tarsus_link: mass 0.067 -> 0.0905228; geometry collision cylinder length=0.055 radius=0.018; visual mesh filename=package://marsdog/meshes/fr_tarsus_link.STL
- link fr_thigh_roll_link: mass 0.087 -> 0.08017506; geometry collision box size=0.01 0.035 0.07; visual mesh filename=package://marsdog/meshes/fr_thigh_roll_link.STL
- link head_pitch_link: mass 0.025 -> 0.78588222
- link head_roll_link: mass 0.274 -> 0.22511155
- link head_yaw_link: mass 0.274 -> 0.22511155
- link neck_pitch_link: mass 0.295 -> 0.24748464
- link rl_calf_link: mass 0.048 -> 0.02748893
- link rl_foot_link: mass 0.005 -> 0.00282686
- link rl_hip_link: mass 0.374 -> 0.40282962
- link rl_tarsus_link: mass 0.032 -> 0.03245619; geometry collision box size=0.014 0.020 0.06; visual mesh filename=package://marsdog/meshes/rl_tarsus_link.STL
- link rl_thigh_link: mass 0.414 -> 0.39029186
- link rr_calf_link: mass 0.048 -> 0.02748893
- link rr_foot_link: mass 0.005 -> 0.00282686
- link rr_hip_link: mass 0.374 -> 0.40282962
- link rr_tarsus_link: mass 0.032 -> 0.03245619
- link rr_thigh_link: mass 0.414 -> 0.38566891
- link waist_pitch_link: mass 1.098 -> 4.23177819; geometry collision box size=0.09 0.10 0.06; collision cylinder length=0.07 radius=0.032
- link waist_roll_link: mass 0.337 -> 0.35780146
- link waist_yaw_link: mass 1.264 -> 1.28140701
Joints:
- removed joint imu_joint
- removed joint tail10_pitch_joint
- removed joint tail10_yaw_joint
- removed joint tail11_pitch_joint
- removed joint tail11_yaw_joint
- removed joint tail12_pitch_joint
- removed joint tail12_yaw_joint
- removed joint tail1_pitch_joint
- removed joint tail1_yaw_joint
- removed joint tail2_pitch_joint
- removed joint tail2_yaw_joint
- removed joint tail3_pitch_joint
- removed joint tail3_yaw_joint
- removed joint tail4_pitch_joint
- removed joint tail4_yaw_joint
- removed joint tail5_pitch_joint
- removed joint tail5_yaw_joint
- removed joint tail6_pitch_joint
- removed joint tail6_yaw_joint
- removed joint tail7_pitch_joint
- removed joint tail7_yaw_joint
- removed joint tail8_pitch_joint
- removed joint tail8_yaw_joint
- removed joint tail9_pitch_joint
- removed joint tail9_yaw_joint
- added joint tail_pitch_joint: type revolute, parent tail_yaw_link, child tail_pitch_link, origin xyz=-0.016782 0 0 rpy=0 0 0, axis 1 0 0, limit lower=-0.3 upper=0.3 effort=6 velocity=10.472
- added joint tail_yaw_joint: type revolute, parent base_link, child tail_yaw_link, origin xyz=-0.16074 0 0.014415 rpy=0 -0.24435 0, axis 0 1 0, limit lower=-0.3 upper=0.3 effort=6 velocity=10.472
- joint fl_calf_joint: axis 0 1 0.001365 -> 0 1 0; origin xyz=0.0235 0.0034955 -0.069995 rpy=0 0 0 -> xyz=0.0204999999999997 0.00849999999999988 -0.0899999999999999 rpy=0 0 0
- joint fl_foot_joint: origin xyz=0 -0.005449 -0.051948 rpy=0 0 0 -> xyz=0 -0.002019916666668 -0.0591902329339155 rpy=0 0 0
- joint fl_hip_pitch_joint: axis 0 1 0.001365 -> 0 1 0; origin xyz=0.11134 0.040867 -0.085936 rpy=0 0 0 -> xyz=0.111344294340592 0.0412499999999985 -0.0819915230487584 rpy=0 0 0
- joint fl_tarsus_joint: axis 0 1 0.001365 -> 0 1 0; limit lower=-1.49 upper=0.03 effort=0.4119 velocity=9.9484 -> lower=-0.03 upper=1.49 effort=0.4119 velocity=9.9484; origin xyz=0.0040403 -0.0022336 -0.12194 rpy=0 0 0 -> xyz=0 -0.0129931382700103 -0.11088651657851 rpy=0 0 0
- joint fl_thigh_roll_joint: axis 0.99966 3.5842E-05 0.026258 -> 1 0 0; origin xyz=-0.0205 0.028 3.8219E-05 rpy=0 0 0 -> xyz=-0.0204999999999978 0.0255000000000006 0 rpy=0 0 0
- joint fr_calf_joint: axis 0 -1 -0.001365 -> 0 1 0; limit lower=-1.93 upper=1.82 effort=6 velocity=10.472 -> lower=-1.82 upper=1.93 effort=6 velocity=10.472; origin xyz=0.02533 -0.0033053 -0.069363 rpy=0 0 0 -> xyz=0.0204999999999999 -0.00849999999999999 -0.0900000000000001 rpy=0 0 0
- joint fr_foot_joint: origin xyz=0 0.0055908 -0.051933 rpy=0 0 0 -> xyz=-0.00112547900491583 0.00201991666666686 -0.0591795316961916 rpy=0 0.0190157527794673 0
- joint fr_hip_pitch_joint: axis 0 -1 -0.001365 -> 0 1 0; limit lower=-0.97 upper=3.14159265358979 effort=17 velocity=32.9867 -> lower=-3.14159265358979 upper=0.97 effort=17 velocity=32.9867; origin xyz=0.11134 -0.040633 -0.086047 rpy=0 0 0 -> xyz=0.111344294340584 -0.0412500000000016 -0.0819915230487582 rpy=0 0 0
- joint fr_tarsus_joint: axis 0 -1 -0.001365 -> 0 1 0; origin xyz=0.0055464 0.0025664 -0.12187 rpy=0 0 0 -> xyz=0 0.0129931382700104 -0.11088651657851 rpy=0 0 0
- joint fr_thigh_roll_joint: axis 0.99966 -3.5842E-05 0.026258 -> 1 0 0; origin xyz=-0.020493 -0.027999 -0.00057652 rpy=0 0 0 -> xyz=-0.020499999999996 -0.0254999999999991 0 rpy=0 0 0
- joint head_pitch_joint: origin xyz=-0.0145282626 -0.0215314491 0.0289972420 rpy=0 0.56570 0 -> xyz=0 -0.012999999999996 0.0299999999999988 rpy=0 0.610865238198016 0
- joint head_roll_joint: axis -1 0.00073162 0 -> 1 0 0; origin xyz=0.067501 -0.02831 0.042889 rpy=0 -0.56569 0 -> xyz=0.062255555366079 -0.0291999999994765 0.0435918091625143 rpy=0 -0.610865238198017 0
- joint head_yaw_joint: origin xyz=0.015514 0.0010134 0.014495 rpy=0 0 0 -> xyz=0.0299999999999988 0 0.013 rpy=0 0 0
- joint neck_pitch_joint: origin xyz=0.063536 0.031281 -0.022505 rpy=0 0 0 -> xyz=0.0634999999999999 0.0282499999999988 -0.0185 rpy=0 0 0
- joint rl_calf_joint: axis 0 -1 -0.001365 -> 0 1 0; limit lower=-1.56 upper=0 effort=14 velocity=32.9867 -> lower=0 upper=1.56 effort=14 velocity=32.9867; origin xyz=0.023309 0.0090594 -0.11679 rpy=0 0 0 -> xyz=0.00815055529011946 0.00790000000000006 -0.11883017880998 rpy=0 0 0
- joint rl_foot_joint: limit lower=-3.14159265358979 upper=3.14159265358979 effort=100 velocity=10 -> (none); origin xyz=0.01159 0.010411 -0.061956 rpy=0 0 0 -> xyz=0.0029939 0.011326 -0.058227 rpy=0 -0.11813 0
- joint rl_hip_joint: axis 1 -0.00046685 0 -> 1 0 0; origin xyz=-0.041722 0.0335 -0.015186 rpy=-0.0014526 -0.34907 0.00049681 -> xyz=-0.0530871685740839 0.0335004012032589 -0.0306494525501697 rpy=0 -0.523598775548837 0
- joint rl_tarsus_joint: axis 0 -1 -0.001365 -> 0 1 0; origin xyz=-0.01875 0.00010616 -0.077772 rpy=0 0 0 -> xyz=-0.038105 5E-05 -0.070342 rpy=0 0 0
- joint rl_thigh_joint: axis 0 1 0.001365 -> 0 1 0; origin xyz=-0.046282 0.039422 5.0587E-05 rpy=0 0.34907 0 -> xyz=-0.047 0.0394 0 rpy=1.309E-05 0.5236 0
- joint rr_calf_joint: axis 0 1 0.001365 -> 0 1 0; origin xyz=0.022904 -0.0087404 -0.1169 rpy=0 0 0 -> xyz=0.00815055529007039 -0.00789999999999996 -0.118830178809943 rpy=0 0 0
- joint rr_foot_joint: origin xyz=0.011375 -0.010242 -0.062024 rpy=0 0 0 -> xyz=0.00299391845062902 -0.0113262512375831 -0.0582274450635127 rpy=0 -0.11812507471832 0
- joint rr_hip_joint: axis 1 -0.00046685 0 -> 1 0 0; origin xyz=-0.041722 -0.0335 -0.015186 rpy=-0.0014526 -0.34907 0.00049681 -> xyz=-0.053087 -0.0335 -0.03065 rpy=0 -0.5236 0
- joint rr_tarsus_joint: axis 0 1 0.001365 -> 0 1 0; origin xyz=-0.019514 0 -0.077584 rpy=0 0 0 -> xyz=-0.0381047330872525 -4.99999999993422E-05 -0.0703422299642889 rpy=0 0 0
- joint rr_thigh_joint: axis 0 -1 -0.001365 -> 0 1 0; limit lower=-1.77 upper=0.71 effort=14 velocity=32.9867 -> lower=-0.71 upper=1.77 effort=14 velocity=32.9867; origin xyz=-0.046318 -0.039378 -5.0537E-05 rpy=0 0.34907 0 -> xyz=-0.0470000000000001 -0.0393999999974683 0 rpy=1.30899691641225E-05 0.523598775561203 0
- joint waist_pitch_joint: axis 0 1 0.001365 -> 0 1 0; origin xyz=0.0415 -0.0235 0 rpy=0 0 0 -> xyz=0.0450000000000001 -0.024 0 rpy=0 0 0
- joint waist_roll_joint: origin xyz=0.055059 0 0.028279 rpy=-0.001365 0 0 -> xyz=0.0455 0 0 rpy=0 0 0
- joint waist_yaw_joint: axis 0 -0.001365 1 -> 0 0 1; origin xyz=0.0635 0.023463 0.026782 rpy=0 0 0 -> xyz=0.0634999999999956 0.0239999999999988 0.0227500000000019 rpy=0 0 0
